File: eagle/DSKY/debouncer_4x.brd (EAGLE design)
At the start: 160 x 100 mm, 11 parts

Commit message: added gitignore file
Parts:
- moved C101 41.8 mm to (8.40, 27.2)
- moved C102 41.8 mm to (6.00, 21.4)
- moved C103 41.8 mm to (6.00, 15.0)
- moved C104 41.8 mm to (9.00, 9.80)
- moved C105 41.8 mm to (21.6, 30.4)
- moved C106 41.8 mm to (21.6, 7.20)
- moved IC101 41.8 mm to (21.6, 30.4)
- moved IC102 41.8 mm to (21.6, 7.20)
- moved RN101 41.8 mm to (20.4, 22.6)
- moved RN102 41.8 mm to (20.4, 15.0)
- moved RN103 41.8 mm to (20.4, 18.8)
Other:
- board outline removed
